File: v1/v1.brd (EAGLE design)
At the start: 101.3 x 80 mm, 19 parts, among them J1 ATX24RH, J2 24VAC, Q1 TIP120, Q2 TIP120, Q3 TIP120, Q4 TIP120, Q5 TIP120, Q6 TIP120, U1 ARDUINO-MEGAFULL

Commit message: last
more changes to come
Connections:
- removed net +5V_EXT: OK1.5, OK2.5, OK3.5, OK4.5, OK5.5
- removed net N$19: J1.23
- removed net N$29: J1.22
- removed net N$59: J1.1
- removed net PIN2: U1.2
- removed net PIN3: U1.3
- removed net PIN4: U1.4
- removed net PIN5: U1.5
- removed net PIN6: U1.6
- removed net PIN7: U1.7
- removed net PIN8: U1.8
- removed net PIN9: U1.9
- new net B$1: J1.22, J1.23, OK1.5, OK2.5, OK3.5, OK4.5, OK5.5
- new net B$2: U$1.1, U$1.2, U$1.3, U$1.4, U$1.5, U$1.6, U$1.7, U$1.8, U1.2, U1.3, U1.4, U1.5, U1.6, U1.7, U1.8, U1.9
- net 3V3_MEGA: now also J1.1
Changed lines of the file:
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@@
 <contactref element="U1" pad="45"/>
-</signal>
-<signal name="+5V_EXT">
-<contactref element="OK1" pad="5"/>
-<contactref element="OK2" pad="5"/>
-<contactref element="OK3" pad="5"/>
-<contactref element="OK4" pad="5"/>
-<contactref element="OK5" pad="5"/>
-<wire x1="-27.94" y1="90.17" x2="-17.78" y2="90.17" width="0" layer="19" extent="1-1"/>
-<wire x1="-38.1" y1="90.17" x2="-27.94" y2="90.17" width="0" layer="19" extent="1-1"/>
-<wire x1="-96.52" y1="66.04" x2="-86.36" y2="66.04" width="0" layer="19" extent="1-1"/>
-<wire x1="-86.36" y1="66.04" x2="-38.1" y2="90.17" width="0" layer="19" extent="1-1"/>
 </signal>
 <signal name="N$2">
@@
 <contactref element="U1" pad="3.3V"/>
 <contactref element="Q6" pad="C"/>
-<wire x1="-76.2" y1="57.15" x2="36.83" y2="20.32" width="0" layer="19" extent="1-1"/>
+<contactref element="J1" pad="1"/>
+<wire x1="-76.2" y1="57.15" x2="-53.1" y2="-7.94" width="0" layer="19" extent="1-1"/>
+<wire x1="36.83" y1="20.32" x2="-53.1" y2="-7.94" width="0" layer="19" extent="1-1"/>
 </signal>
 <signal name="S_FAN">
@@
 <contactref element="MISTER_RELAY" pad="4"/>
 </signal>
-<signal name="PIN2">
-<contactref element="U1" pad="2"/>
-</signal>
-<signal name="PIN3">
-<contactref element="U1" pad="3"/>
-</signal>
-<signal name="PIN4">
-<contactref element="U1" pad="4"/>
-</signal>
-<signal name="PIN5">
-<contactref element="U1" pad="5"/>
-</signal>
-<signal name="PIN6">
-<contactref element="U1" pad="6"/>
-</signal>
-<signal name="PIN7">
-<contactref element="U1" pad="7"/>
-</signal>
-<signal name="PIN8">
-<contactref element="U1" pad="8"/>
-</signal>
-<signal name="PIN9">
-<contactref element="U1" pad="9"/>
-</signal>
 <signal name="N$20">
 <contactref element="U1" pad="10"/>
@@
 <contactref element="J1" pad="18"/>
 </signal>
-<signal name="N$19">
-<contactref element="J1" pad="23"/>
-</signal>
-<signal name="N$29">
-<contactref element="J1" pad="22"/>
-</signal>
 <signal name="N$56">
 <contactref element="J1" pad="21"/>
@@
 <contactref element="J1" pad="6"/>
 </signal>
-<signal name="N$59">
-<contactref element="J1" pad="1"/>
-</signal>
 <signal name="N$60">
 <contactref element="J1" pad="2"/>
@@
 <contactref element="J1" pad="14"/>
 </signal>
+<signal name="B$1">
+<contactref element="OK3" pad="5"/>
+<contactref element="OK5" pad="5"/>
+<contactref element="OK4" pad="5"/>
+<contactref element="OK2" pad="5"/>
+<contactref element="OK1" pad="5"/>
+<contactref element="J1" pad="23"/>
+<contactref element="J1" pad="22"/>
+<wire x1="-90.9" y1="-2.44" x2="-95.1" y2="-2.44" width="0" layer="19" extent="1-1"/>
+<wire x1="-96.52" y1="66.04" x2="-95.1" y2="-2.44" width="0" layer="19" extent="1-1"/>
+<wire x1="-86.36" y1="66.04" x2="-96.52" y2="66.04" width="0" layer="19" extent="1-1"/>
+<wire x1="-38.1" y1="90.17" x2="-86.36" y2="66.04" width="0" layer="19" extent="1-1"/>
+<wire x1="-27.94" y1="90.17" x2="-38.1" y2="90.17" width="0" layer="19" extent="1-1"/>
+<wire x1="-17.78" y1="90.17" x2="-27.94" y2="90.17" width="0" layer="19" extent="1-1"/>
+</signal>
+<signal name="B$2">
+<contactref element="U1" pad="2"/>
+<contactref element="U1" pad="3"/>
+<contactref element="U1" pad="4"/>
+<contactref element="U1" pad="5"/>
+<contactref element="U1" pad="6"/>
+<contactref element="U1" pad="7"/>
+<contactref element="U1" pad="8"/>
+<contactref element="U1" pad="9"/>
+<contactref element="U$1" pad="8"/>
+<contactref element="U$1" pad="7"/>
+<contactref element="U$1" pad="6"/>
+<contactref element="U$1" pad="5"/>
+<contactref element="U$1" pad="4"/>
+<contactref element="U$1" pad="3"/>
+<contactref element="U$1" pad="2"/>
+<contactref element="U$1" pad="1"/>
+<wire x1="57.15" y1="68.58" x2="59.69" y2="68.58" width="0" layer="19" extent="1-1"/>
+<wire x1="54.61" y1="68.58" x2="57.15" y2="68.58" width="0" layer="19" extent="1-1"/>
+<wire x1="52.07" y1="68.58" x2="54.61" y2="68.58" width="0" layer="19" extent="1-1"/>
+<wire x1="49.53" y1="68.58" x2="52.07" y2="68.58" width="0" layer="19" extent="1-1"/>
+<wire x1="46.99" y1="68.58" x2="49.53" y2="68.58" width="0" layer="19" extent="1-1"/>
+<wire x1="42.926" y1="68.58" x2="46.99" y2="68.58" width="0" layer="19" extent="1-1"/>
+<wire x1="40.386" y1="68.58" x2="42.926" y2="68.58" width="0" layer="19" extent="1-1"/>
+<wire x1="-106.045" y1="-3.81" x2="40.386" y2="68.58" width="0" layer="19" extent="1-1"/>
+<wire x1="-108.585" y1="-3.81" x2="-106.045" y2="-3.81" width="0" layer="19" extent="1-1"/>
+<wire x1="-111.125" y1="-3.81" x2="-108.585" y2="-3.81" width="0" layer="19" extent="1-1"/>
+<wire x1="-113.665" y1="-3.81" x2="-111.125" y2="-3.81" width="0" layer="19" extent="1-1"/>
+<wire x1="-114.935" y1="-6.35" x2="-113.665" y2="-3.81" width="0" layer="19" extent="1-1"/>
+<wire x1="-112.395" y1="-6.35" x2="-114.935" y2="-6.35" width="0" layer="19" extent="1-1"/>
+<wire x1="-109.855" y1="-6.35" x2="-112.395" y2="-6.35" width="0" layer="19" extent="1-1"/>
+<wire x1="-107.315" y1="-6.35" x2="-109.855" y2="-6.35" width="0" layer="19" extent="1-1"/>
+</signal>
 </signals>
