File: v1/v1.sch (EAGLE design)
At the start: 15 parts, among them Q1 TIP120, Q2 TIP120, Q3 TIP120, Q4 TIP120, Q5 TIP120, Q6 TIP120, U1 ARDUINO-MEGAFULL

Commit message: Framed
Added a frame, some connectors and resistors on signalpins. These should
have a pulldown to gnd aswell.
Parts:
- added J1: ATX24RH, SparkFun-Connectors:ATX24RH
- added J2: 24VAC, SparkFun-Connectors:POWER_JACKSLT
- added JP1: M025MM, SparkFun-Connectors:M025MM
- added U$1: RJ45-8PTH, SparkFun-Connectors:RJ45-8PTH
Connections:
- net +24VAC renamed 24VAC
- net N$19 renamed PIN9
- new net +12VCC: Q5.C
- new net N$10: U1.24
- new net N$11: U1.23
- new net N$13: U1.25
- new net N$14: U1.26
- new net N$16: U1.27
- new net N$17: U1.28
- new net N$19: J1.5V@4
- new net N$3: J1.GND@7
- new net N$4: U1.A0(RX0)
- new net N$47: U1.29
- new net N$48: U1.GND@0
- new net N$49: U1.GND@1
- new net N$50: U1.GND@3
- new net N$51: U1.GND@2
- new net N$52: U1.GND@4
- new net N$53: U1.0(RX0)
- new net N$54: U1.1(TX0)
- new net N$55: U1.AREF
- new net N$56: J1.5V@2
- new net N$57: J1.5V@0
- new net N$58: J1.5V@1
- new net N$59: J1.3.3V@0
- new net N$60: J1.3.3V@1
- new net N$61: J1.3.3V@3
- new net N$62: J1.12V@0
- new net N$63: J1.12V@1
- new net N$64: J1.-12V
- new net N$7: U1.22
- net DEVICE_SUPPLY: no longer Q5.C
- net GND: now also C1.-, U1.12
- net N$29: now also J1.5V@3; no longer U1.12
- net N$5: now also J1.GND@6; no longer U1.5V@0
- net N$6: now also J1.GND@5; no longer U1.5V@1
- net S_IN: now also C1.+
Other:
- note added: "Vi må ha RCfiltere og noen steder"
- moved on the sheet: C1, LED1, MISTER_RELAY, OK1, OK2, OK3, OK4, OK5, Q1, Q2, Q3, Q4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

Commit message: Last
Uppdateted text
Other:
- note added: "3.01"
- note added: "Kristebo"
- note added: "Krydderino"
Changed lines of the file:
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@@
 <text x="-167.64" y="233.68" size="6.4516" layer="97">LED_DRIVER</text>
 <text x="114.3" y="139.7" size="1.778" layer="91">Vi må ha RCfiltere og noen steder</text>
+<text x="124.46" y="35.56" size="1.778" layer="91">Krydderino</text>
+<text x="127" y="30.48" size="1.778" layer="91">3.01</text>
+<text x="132.08" y="20.32" size="1.778" layer="91">Kristebo</text>
 </plain>
 <instances>

Commit message: last
more changes to come
Connections:
- removed net +5V_EXT: OK1.COL, OK2.COL, OK3.COL, OK4.COL, OK5.COL
- removed net N$19: J1.5V@4
- removed net N$29: J1.5V@3
- removed net N$56: J1.5V@2
- removed net N$57: J1.5V@0
- removed net N$58: J1.5V@1
- removed net N$59: J1.3.3V@0
- removed net PIN2: U1.2
- removed net PIN3: U1.3
- removed net PIN4: U1.4
- removed net PIN5: U1.5
- removed net PIN6: U1.6
- removed net PIN7: U1.7
- removed net PIN8: U1.8
- removed net PIN9: U1.9
- new net B$1: J1.5V@0, J1.5V@1, J1.5V@2, J1.5V@3, J1.5V@4, OK1.COL, OK2.COL, OK3.COL, OK4.COL, OK5.COL
- new net B$2: U$1.1, U$1.2, U$1.3, U$1.4, U$1.5, U$1.6, U$1.7, U$1.8, U1.2, U1.3, U1.4, U1.5, U1.6, U1.7, U1.8, U1.9
- net 3V3_MEGA: now also J1.3.3V@0
